File: pcb/digisax.kicad_pcb (KiCad board)
At the start: 2 copper layers, 48 parts, among them SW1 RotaryEncoder_Switch, U1 ER_OLEDM0.91_1x-I2C, U2 MPXV7007, U3 MCP3221, U4 TLV320DAC3100_breakout, U5 ESP32-S3

Commit message: added all symbols :D
Parts:
- added BT1: Battery, digisax_stuff:5V0_terminal, F.Cu at (-76.7, 147.1)
- added C1: 470pF, Capacitor_THT:C_Disc_D4.7mm_W2.5mm_P5.00mm, F.Cu at (-41.0, 25.8)
- added C2: 100nF, Capacitor_THT:C_Disc_D4.7mm_W2.5mm_P5.00mm, F.Cu at (-49.2, 25.8)
- added C3: 100nF, Capacitor_THT:C_Disc_D4.7mm_W2.5mm_P5.00mm, F.Cu at (-56.3, 36.4)
- added C4: 470uF, Capacitor_THT:CP_Radial_D6.3mm_P2.50mm, F.Cu at (-24.9, 14.1)
- moved U3 406.1 mm to (412.6, -195.6)
- moved SW1 313.7 mm to (-111.5, 86.8)
- moved U5 305.1 mm to (-112.7, 156.9)
- moved U4 249.7 mm to (-103.1, 54.5)
- moved D10 217.5 mm to (-55.6, -27.0)
- moved D11 217.5 mm to (-55.6, -23.5)
- moved D12 217.5 mm to (-55.6, -19.9)
- moved D13 217.5 mm to (-55.6, -16.4)
- moved D14 217.5 mm to (-55.6, -12.8)
- moved D8 217.5 mm to (-55.6, -34.1)
- moved D9 217.5 mm to (-55.6, -30.6)
- moved D1 217.5 mm to (-66.4, -34.1)
- moved D15 217.5 mm to (-44.8, -34.1)
- moved D16 217.5 mm to (-44.8, -30.6)
- moved D17 217.5 mm to (-44.8, -27.0)
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
Commit message: new switch models.. yeah
Parts:
- removed key_8VE1, key_BF1, key_CS1, key_DS1, key_GS1, key_LBF1, key_LS1, key_LS2, key_LS3: SW_Push, Button_Switch_Keyboard:SW_Cherry_MX_1.00u_PCB
- added key_Bflat1: SW_Push, digisax_stuff:slim_switch, F.Cu at (213.0, 140.0)
- added key_Csharp1: SW_Push, digisax_stuff:slim_switch, F.Cu at (213.0, 155.1)
- added key_Dsharp1: SW_Push, digisax_stuff:slim_switch, F.Cu at (213.0, 170.2)
- added key_Gsharp1: SW_Push, digisax_stuff:slim_switch, F.Cu at (228.1, 140.0)
- added key_LBflat1: SW_Push, digisax_stuff:slim_switch, F.Cu at (228.1, 155.1)
- added key_Lside1: SW_Push, digisax_stuff:slim_switch, F.Cu at (228.1, 170.2)
- added key_Lside2: SW_Push, digisax_stuff:slim_switch, F.Cu at (243.2, 140.0)
- added key_Lside3: SW_Push, digisax_stuff:slim_switch, F.Cu at (243.2, 155.1)
- added key_octave1: SW_Push, digisax_stuff:slim_switch, F.Cu at (243.2, 170.2)
- key_C1, key_L1, key_L2, key_L3, key_LB1, key_R1, key_R2, key_R3, key_RS1, key_RS2, key_RS3: footprint Button_Switch_Keyboard:SW_Cherry_MX_1.00u_PCB -> digisax_stuff:slim_switch
- key_fork1: renamed from key_FORK1; footprint Button_Switch_Keyboard:SW_Cherry_MX_1.00u_PCB -> digisax_stuff:slim_switch
- moved U3 629.5 mm to (-153.4, 79.8)
- moved key_LB1 287.1 mm to (357.8, 188.2)
- moved key_L2 145.0 mm to (213.5, 51.9)
- moved key_C1 144.5 mm to (110.5, 236.0)
- moved key_RS3 130.0 mm to (58.9, 220.9)
- moved key_RS2 123.5 mm to (57.9, 198.2)
- moved key_RS1 120.6 mm to (57.4, 179.8)
- moved key_L1 95.1 mm to (161.5, 41.9)
- moved key_fork1 67.7 mm to (104.8, 164.0)
- moved key_L3 65.6 mm to (131.7, 79.5)
- moved key_R2 50.5 mm to (132.2, 160.3)
- moved key_R1 45.9 mm to (131.8, 137.4)
- moved key_R3 40.8 mm to (134.4, 181.9)

Commit message: switch placement according to irl sax
Parts:
- removed key_RS1, key_RS2, key_RS3: SW_Push, digisax_stuff:slim_switch
- added key_Rside1: SW_Push, digisax_stuff:slim_switch, F.Cu at (101.5, 125.5)
- added key_Rside2: SW_Push, digisax_stuff:slim_switch, F.Cu at (101.5, 147.5)
- added key_Rside3: SW_Push, digisax_stuff:slim_switch, F.Cu at (101.4, 169.5)
- key_octave1: moved to B.Cu
- moved key_LB1 146.7 mm to (218.8, 141.0)
- moved key_octave1 140.0 mm to (189.4, 41.0), turned to 180 degrees
- moved key_Lside1 116.5 mm to (280.1, 66.0)
- moved key_Dsharp1 110.4 mm to (118.4, 227.0)
- moved key_Lside2 92.5 mm to (252.1, 48.0)
- moved key_Lside3 75.2 mm to (240.1, 80.0)
- moved key_L3 68.5 mm to (185.5, 121.9)
- moved key_L2 65.4 mm to (174.4, 104.4)
- moved key_Bflat1 64.8 mm to (174.4, 88.0)
- moved key_R2 43.7 mm to (172.4, 177.5)
- moved key_fork1 43.3 mm to (140.4, 188.5)
- moved key_R3 39.0 mm to (165.4, 205.5)
- moved key_R1 36.2 mm to (167.5, 143.5)
- moved key_L1 32.2 mm to (174.4, 71.4)
- moved key_Csharp1 26.4 mm to (235.3, 141.0)
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
Commit message: added headers to schem
Parts:
- U2: moved to B.Cu
- moved D18 374.5 mm to (278.9, 164.8)
- moved D19 374.5 mm to (278.9, 168.4)
- moved D20 374.5 mm to (278.9, 171.9)
- moved D21 374.5 mm to (278.9, 175.5)
- moved U5 321.2 mm to (198.7, 235.8)
- moved D12 321.1 mm to (198.9, 175.9)
- moved D13 321.1 mm to (198.9, 179.4)
- moved D14 321.1 mm to (198.9, 183.0)
- moved D15 317.9 mm to (255.4, 70.5)
- moved D17 317.2 mm to (255.4, 75.5)
- moved D16 315.2 mm to (255.4, 65.5)
- moved D5 294.6 mm to (90.4, 229.4)
- moved D6 294.6 mm to (90.4, 233.0)
- moved D10 270.1 mm to (189.5, 86.5)
- moved D11 270.1 mm to (189.5, 90.0)
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
Commit message: more kcal burnt on pcb
Parts:
- added J1: Conn_01x04_Pin, digisax_stuff:pad_1x4, F.Cu at (217.8, 127.1)
- added J2: Conn_01x04_Pin, digisax_stuff:pad_1x4, F.Cu at (166.0, 143.7)
- added J3: Conn_01x05_Pin, digisax_stuff:pad_1x5, F.Cu at (215.0, 190.1)
- added J4: Conn_01x05_Pin, digisax_stuff:pad_1x5, F.Cu at (163.5, 197.9)
- added J5: Conn_01x04_Pin, digisax_stuff:pad_1x4, F.Cu at (74.4, 201.1)
- added J6: Conn_01x04_Pin, digisax_stuff:pad_1x4, F.Cu at (134.8, 203.1)
- added J7: Conn_01x03_Pin, digisax_stuff:pad_1x3, F.Cu at (45.0, 286.1)
- added J8: Conn_01x03_Pin, digisax_stuff:pad_1x3, F.Cu at (126.7, 256.9)
- SW1, U1, U4: moved to B.Cu
- moved C3 358.3 mm to (172.2, 312.4)
- moved U4 356.4 mm to (154.0, 301.3), turned to 180 degrees
- moved C4 350.5 mm to (160.7, 311.4)
- moved SW1 331.0 mm to (175.0, 252.5), turned to 180 degrees
- moved BT1 291.3 mm to (169.0, 303.5)
- moved U1 266.3 mm to (165.8, 243.1), turned to 0 degrees
- moved C2 216.5 mm to (126.4, 152.5)
- moved C1 213.4 mm to (121.3, 164.3)
- moved U2 210.7 mm to (145.1, 163.1)
- moved U3 206.0 mm to (145.8, 163.6)
- moved D11 85.6 mm to (169.5, 173.3), turned to 180 degrees
- moved D10 77.2 mm to (142.3, 147.6), turned to 90 degrees
- moved D14 75.6 mm to (144.9, 235.9)
- moved U5 71.3 mm to (142.3, 279.6), turned to -90 degrees
- moved key_C1 70.9 mm to (60.2, 287.0)
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Connections:
- D1 pad 1: key_R1 -> key_row1
- D10 pad 1: key_R4 -> key_row3
- D11 pad 1: key_R5 -> key_row4
- D12 pad 1: key_R7 -> key_row5
- D13 pad 1: key_R8 -> key_row6
- D14 pad 1: key_R9 -> key_row7
- D15 pad 1: key_R1 -> Net-(D15-K)
- D16 pad 1: key_R2 -> Net-(D16-K)
- D17 pad 1: key_R4 -> Net-(D17-K)
- D18 pad 1: key_R5 -> Net-(D18-K)
- D19 pad 1: key_R7 -> Net-(D19-K)
- D2 pad 1: key_R2 -> Net-(D2-K)
- D20 pad 1: key_R8 -> Net-(D20-K)
- D21 pad 1: key_R9 -> Net-(D21-K)
- D3 pad 1: key_R4 -> Net-(D3-K)
- D4 pad 1: key_R5 -> Net-(D4-K)
- D5 pad 1: key_R7 -> Net-(D5-K)
- D6 pad 1: key_R8 -> Net-(D6-K)
- D7 pad 1: key_R9 -> key_row7
- D8 pad 1: key_R1 -> key_row1
- D9 pad 1: key_R2 -> key_row2
- key_Bflat1 pad 2: key_C2 -> key_col2
- key_C1 pad 2: key_C1 -> Net-(J7-Pin_3)
- key_Csharp1 pad 2: key_C3 -> Net-(J3-Pin_5)
- key_Dsharp1 pad 2: key_C1 -> Net-(J7-Pin_3)
- key_Gsharp1 pad 2: key_C3 -> Net-(J3-Pin_5)
- key_L1 pad 2: key_C2 -> key_col2
- key_L2 pad 2: key_C2 -> key_col2
- key_L3 pad 2: key_C2 -> key_col2
- key_LB1 pad 2: key_C3 -> Net-(J3-Pin_5)
- key_LBflat1 pad 2: key_C3 -> Net-(J3-Pin_5)
- key_Lside1 pad 2: key_C3 -> Net-(J1-Pin_4)
- key_Lside2 pad 2: key_C3 -> Net-(J1-Pin_4)
- key_Lside3 pad 2: key_C3 -> Net-(J1-Pin_4)
- key_R1 pad 2: key_C2 -> key_col2
- key_R2 pad 2: key_C2 -> key_col2
- key_R3 pad 2: key_C2 -> key_col2
- key_Rside1 pad 2: key_C1 -> Net-(J5-Pin_4)
- key_Rside2 pad 2: key_C1 -> Net-(J5-Pin_4)
- key_Rside3 pad 2: key_C1 -> Net-(J5-Pin_4)
- key_fork1 pad 2: key_C1 -> key_col1
- key_octave1 pad 2: key_C1 -> key_col1
Other:
- board outline added: 231.5 x 253.1 mm

Commit message: added barrel jack, sketched board outline
Parts:
- added J9: Barrel_Jack, Connector_BarrelJack:BarrelJack_Horizontal, F.Cu at (146.0, 309.3)
- added REF**: MountingHole_3.2mm_M3, MountingHole:MountingHole_3.2mm_M3, F.Cu at (228.0, 215.0)
- added REF**: MountingHole_3.2mm_M3, MountingHole:MountingHole_3.2mm_M3, F.Cu at (196.0, 148.0)
- added REF**: MountingHole_3.2mm_M3, MountingHole:MountingHole_3.2mm_M3, F.Cu at (132.0, 297.0)
- added REF**: MountingHole_3.2mm_M3, MountingHole:MountingHole_3.2mm_M3, F.Cu at (229.0, 160.0)
- added REF**: MountingHole_3.2mm_M3, MountingHole:MountingHole_3.2mm_M3, F.Cu at (132.0, 253.0)
- added REF**: MountingHole_3.2mm_M3, MountingHole:MountingHole_3.2mm_M3, F.Cu at (172.0, 148.0)
- added REF**: MountingHole_3.2mm_M3, MountingHole:MountingHole_3.2mm_M3, F.Cu at (194.0, 160.0)
- added REF**: MountingHole_3.2mm_M3, MountingHole:MountingHole_3.2mm_M3, F.Cu at (178.0, 160.0)
- added REF**: MountingHole_3.2mm_M3, MountingHole:MountingHole_3.2mm_M3, F.Cu at (194.0, 215.0)
- added REF**: MountingHole_3.2mm_M3, MountingHole:MountingHole_3.2mm_M3, F.Cu at (121.0, 297.0)
- added REF**: MountingHole_3.2mm_M3, MountingHole:MountingHole_3.2mm_M3, F.Cu at (95.0, 297.0)
- added REF**: MountingHole_3.2mm_M3, MountingHole:MountingHole_3.2mm_M3, F.Cu at (95.0, 253.0)
- added REF**: MountingHole_3.2mm_M3, MountingHole:MountingHole_3.2mm_M3, F.Cu at (181.0, 215.0)
- added REF**: MountingHole_3.2mm_M3, MountingHole:MountingHole_3.2mm_M3, F.Cu at (133.0, 198.0)
- added REF**: MountingHole_3.2mm_M3, MountingHole:MountingHole_3.2mm_M3, F.Cu at (196.0, 89.0)
- added REF**: MountingHole_3.2mm_M3, MountingHole:MountingHole_3.2mm_M3, F.Cu at (172.0, 89.0)
- added REF**: MountingHole_3.2mm_M3, MountingHole:MountingHole_3.2mm_M3, F.Cu at (102.0, 198.0)
- added REF**: MountingHole_3.2mm_M3, MountingHole:MountingHole_3.2mm_M3, F.Cu at (120.0, 127.0)
- added REF**: MountingHole_3.2mm_M3, MountingHole:MountingHole_3.2mm_M3, F.Cu at (247.0, 89.0)
- added REF**: MountingHole_3.2mm_M3, MountingHole:MountingHole_3.2mm_M3, F.Cu at (120.0, 198.0)
- added REF**: MountingHole_3.2mm_M3, MountingHole:MountingHole_3.2mm_M3, F.Cu at (102.0, 127.0)
- added REF**: MountingHole_3.2mm_M3, MountingHole:MountingHole_3.2mm_M3, F.Cu at (247.0, 148.0)
- added REF**: MountingHole_3.2mm_M3, MountingHole:MountingHole_3.2mm_M3, F.Cu at (133.0, 127.0)
- added REF**: MountingHole_3.2mm_M3, MountingHole:MountingHole_3.2mm_M3, F.Cu at (120.0, 253.0)
- moved key_Rside3 52.0 mm to (110.5, 185.0)
- moved J5 52.0 mm to (121.8, 179.7)
- moved key_Rside1 52.0 mm to (110.6, 141.0)
- moved key_Rside2 52.0 mm to (110.6, 163.0)
- moved D2 50.7 mm to (122.0, 148.0), turned to 90 degrees
- moved D6 50.1 mm to (93.3, 263.7)
- moved D5 50.1 mm to (93.3, 260.2)
- moved J7 50.1 mm to (94.9, 282.2)
- moved key_C1 50.1 mm to (110.1, 283.1)
- moved key_Dsharp1 50.1 mm to (113.1, 265.4)
- moved D4 38.5 mm to (107.1, 152.2)
- moved D3 32.8 mm to (107.1, 174.1)
- moved C4 26.8 mm to (184.5, 299.0)
- moved J8 25.7 mm to (132.0, 282.0)
- moved U4 25.4 mm to (179.4, 301.8)
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Connections:
- U5 pad 10: key_R5 -> key_row4
- U5 pad 11: key_R7 -> key_row5
- U5 pad 12: key_R8 -> key_row6
- U5 pad 15: key_R9 -> key_row7
- U5 pad 16: key_C1 -> key_col1
- U5 pad 17: key_C2 -> key_col2
- U5 pad 18: key_C3 -> key_col3
- U5 pad 7: key_R1 -> key_row1
- U5 pad 8: key_R2 -> key_row2
- U5 pad 9: key_R4 -> key_row3
Other:
- board size 231.5 x 253.1 mm -> 160 x 250 mm

Commit message: had a go at routing
Parts:
- moved C3 59.1 mm to (146.0, 262.5), turned to 180 degrees
- moved C4 50.1 mm to (151.3, 261.5)
- moved D20 40.5 mm to (191.7, 206.5)
- moved D3 23.8 mm to (115.8, 152.0), turned to 180 degrees
- moved D4 23.5 mm to (115.8, 174.0), turned to 180 degrees
- moved D18 9.55 mm to (219.0, 169.2), turned to -90 degrees
- moved D19 7.41 mm to (226.0, 206.5), turned to 90 degrees
- moved J1 6.81 mm to (195.5, 123.8)
- moved C2 6.02 mm to (139.5, 153.5), turned to 180 degrees
Connections:
- U5 pad 19: unconnected-(U5-GPIO13-Pad19) -> I2C_SDA
- U5 pad 20: unconnected-(U5-GPIO14-Pad20) -> I2C_SCL
Routing:
- net +5V: track 0.00 -> 270.4 mm
- net key_col1: track 0.00 -> 244.1 mm
- net key_row1: track 0.00 -> 225.5 mm
- net key_row5: track 0.00 -> 164.4 mm
- net key_col3: track 0.00 -> 79.2 mm
- net Net-(J1-Pin_4): track 0.00 -> 77.1 mm
- net key_col2: track 0.00 -> 67.1 mm
- net key_row6: track 0.00 -> 66.3 mm
- net Net-(J5-Pin_4): track 0.00 -> 64.8 mm
- net key_row7: track 0.00 -> 63.6 mm
- net Net-(J3-Pin_5): track 0.00 -> 61.1 mm
- net key_row3: track 0.00 -> 52.5 mm
- net Net-(D19-K): track 0.00 -> 49.1 mm
- net key_row2: track 0.00 -> 41.0 mm
- net I2C_SDA: track 0.00 -> 37.0 mm
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
Commit message: routed central board in new kicad project
Parts:
- renumbered REF** to h1, REF** to h10, REF** to h11, REF** to h12, REF** to h13, REF** to h14, REF** to h16, REF** to h17, REF** to h18, REF** to h19, REF** to h2, REF** to h20, REF** to h21, REF** to h22, REF** to h23, REF** to h24, REF** to h25, REF** to h3, REF** to h4, REF** to h5, REF** to h6, REF** to h7, REF** to h8, REF** to h9
Changed lines of the file:
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@@
 		(descr "Mounting Hole 3.2mm, M3, no annular, generated by kicad-footprint-generator mountinghole.py")
 		(tags "mountinghole M3")
-		(property "Reference" "REF**"
+		(property "Reference" "h16"
 			(at 0 -4.15 0)
 			(layer "F.SilkS")
@@
 		(descr "Mounting Hole 3.2mm, M3, no annular, generated by kicad-footprint-generator mountinghole.py")
 		(tags "mountinghole M3")
-		(property "Reference" "REF**"
+		(property "Reference" "h22"
 			(at 0 -4.15 0)
 			(layer "F.SilkS")
@@
 		(descr "Mounting Hole 3.2mm, M3, no annular, generated by kicad-footprint-generator mountinghole.py")
 		(tags "mountinghole M3")
-		(property "Reference" "REF**"
+		(property "Reference" "h19"
 			(at 0 -4.15 0)
 			(layer "F.SilkS")
@@
 		(descr "Mounting Hole 3.2mm, M3, no annular, generated by kicad-footprint-generator mountinghole.py")
 		(tags "mountinghole M3")
-		(property "Reference" "REF**"
+		(property "Reference" "h10"
 			(at 0 -4.15 0)
 			(layer "F.SilkS")
@@
 		(descr "Mounting Hole 3.2mm, M3, no annular, generated by kicad-footprint-generator mountinghole.py")
 		(tags "mountinghole M3")
-		(property "Reference" "REF**"
+		(property "Reference" "h21"
 			(at 0 -4.15 0)
 			(layer "F.SilkS")
@@
 		(descr "Mounting Hole 3.2mm, M3, no annular, generated by kicad-footprint-generator mountinghole.py")
 		(tags "mountinghole M3")
-		(property "Reference" "REF**"
+		(property "Reference" "h18"
 			(at 0 -4.15 0)
 			(layer "F.SilkS")
@@
 		(descr "Mounting Hole 3.2mm, M3, no annular, generated by kicad-footprint-generator mountinghole.py")
 		(tags "mountinghole M3")
-		(property "Reference" "REF**"
+		(property "Reference" "h12"
 			(at 0 -4.15 0)
 			(layer "F.SilkS")
@@
 		(descr "Mounting Hole 3.2mm, M3, no annular, generated by kicad-footprint-generator mountinghole.py")
 		(tags "mountinghole M3")
-		(property "Reference" "REF**"
+		(property "Reference" "h2"
 			(at 0 -4.15 0)
 			(layer "F.SilkS")
@@
 		(descr "Mounting Hole 3.2mm, M3, no annular, generated by kicad-footprint-generator mountinghole.py")
 		(tags "mountinghole M3")
-		(property "Reference" "REF**"
+		(property "Reference" "h23"
 			(at 0 -4.15 0)
 			(layer "F.SilkS")
@@
 		(descr "Mounting Hole 3.2mm, M3, no annular, generated by kicad-footprint-generator mountinghole.py")
 		(tags "mountinghole M3")
-		(property "Reference" "REF**"
+		(property "Reference" "h11"
 			(at 0 -4.15 0)
 			(layer "F.SilkS")
@@
 		(descr "Mounting Hole 3.2mm, M3, no annular, generated by kicad-footprint-generator mountinghole.py")
 		(tags "mountinghole M3")
-		(property "Reference" "REF**"
+		(property "Reference" "h8"
 			(at 0 -4.15 0)
 			(layer "F.SilkS")
@@
 		(descr "Mounting Hole 3.2mm, M3, no annular, generated by kicad-footprint-generator mountinghole.py")
 		(tags "mountinghole M3")
-		(property "Reference" "REF**"
+		(property "Reference" "h14"
 			(at 0 -4.15 0)
 			(layer "F.SilkS")
@@
 		(descr "Mounting Hole 3.2mm, M3, no annular, generated by kicad-footprint-generator mountinghole.py")
 		(tags "mountinghole M3")
-		(property "Reference" "REF**"
+		(property "Reference" "h7"
 			(at 0 -4.15 0)
 			(layer "F.SilkS")
@@
 		(descr "Mounting Hole 3.2mm, M3, no annular, generated by kicad-footprint-generator mountinghole.py")
 		(tags "mountinghole M3")
-		(property "Reference" "REF**"
+		(property "Reference" "h3"
 			(at 0 -4.15 0)
 			(layer "F.SilkS")
@@
 		(descr "Mounting Hole 3.2mm, M3, no annular, generated by kicad-footprint-generator mountinghole.py")
 		(tags "mountinghole M3")
-		(property "Reference" "REF**"
+		(property "Reference" "h13"
 			(at 0 -4.15 0)
 			(layer "F.SilkS")
@@
 		(descr "Mounting Hole 3.2mm, M3, no annular, generated by kicad-footprint-generator mountinghole.py")
 		(tags "mountinghole M3")
-		(property "Reference" "REF**"
+		(property "Reference" "h4"
 			(at 0 -4.15 0)
 			(layer "F.SilkS")
@@
 		(descr "Mounting Hole 3.2mm, M3, no annular, generated by kicad-footprint-generator mountinghole.py")
 		(tags "mountinghole M3")
-		(property "Reference" "REF**"
+		(property "Reference" "h17"
 			(at 0 -4.15 0)
 			(layer "F.SilkS")
@@
 		(descr "Mounting Hole 3.2mm, M3, no annular, generated by kicad-footprint-generator mountinghole.py")
 		(tags "mountinghole M3")
-		(property "Reference" "REF**"
+		(property "Reference" "h25"
 			(at 0 -4.15 0)
 			(layer "F.SilkS")
@@
 		(descr "Mounting Hole 3.2mm, M3, no annular, generated by kicad-footprint-generator mountinghole.py")
 		(tags "mountinghole M3")
-		(property "Reference" "REF**"
+		(property "Reference" "h24"
 			(at 0 -4.15 0)
 			(layer "F.SilkS")
@@
 		(descr "Mounting Hole 3.2mm, M3, no annular, generated by kicad-footprint-generator mountinghole.py")
 		(tags "mountinghole M3")
-		(property "Reference" "REF**"
+		(property "Reference" "h6"
 			(at 0 -4.15 0)
 			(layer "F.SilkS")
@@
 		(descr "Mounting Hole 3.2mm, M3, no annular, generated by kicad-footprint-generator mountinghole.py")
 		(tags "mountinghole M3")
-		(property "Reference" "REF**"
+		(property "Reference" "h5"
 			(at 0 -4.15 0)
 			(layer "F.SilkS")
@@
 		(descr "Mounting Hole 3.2mm, M3, no annular, generated by kicad-footprint-generator mountinghole.py")
 		(tags "mountinghole M3")
-		(property "Reference" "REF**"
+		(property "Reference" "h9"
 			(at 0 -4.15 0)
 			(layer "F.SilkS")
@@
 		(descr "Mounting Hole 3.2mm, M3, no annular, generated by kicad-footprint-generator mountinghole.py")
 		(tags "mountinghole M3")
-		(property "Reference" "REF**"
+		(property "Reference" "h1"
 			(at 0 -4.15 0)
 			(layer "F.SilkS")
@@
 		(descr "Mounting Hole 3.2mm, M3, no annular, generated by kicad-footprint-generator mountinghole.py")
 		(tags "mountinghole M3")
-		(property "Reference" "REF**"
+		(property "Reference" "h20"
 			(at 0 -4.15 0)
 			(layer "F.SilkS")
