File: pcb/digisax.kicad_pcb (KiCad board)
At the start: 2 copper layers, 160 x 250 mm, 86 parts, among them J1 Conn_01x04_Pin, J2 Conn_01x04_Pin, J3 Conn_01x05_Pin, J4 Conn_01x05_Pin, J5 Conn_01x04_Pin, J6 Conn_01x04_Pin, J7 Conn_01x03_Pin, J8 Conn_01x03_Pin, J9 Barrel_Jack, SW1 RotaryEncoder_Switch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

Commit message: added silkscreen art
Parts:
- added neck1: MountingHole_3.2mm_M3, MountingHole:MountingHole_3.2mm_M3, F.Cu at (167.5, 77.0)
- added neck2: MountingHole_3.2mm_M3, MountingHole:MountingHole_3.2mm_M3, F.Cu at (167.5, 102.0)
- added neck3: MountingHole_3.2mm_M3, MountingHole:MountingHole_3.2mm_M3, F.Cu at (140.5, 102.0)
- moved D1 30.8 mm to (137.5, 116.6)
- moved BT1 26.1 mm to (158.0, 314.0)
Routing:
- net key_col1: track 244.1 -> 0.00 mm
- net key_row1: track 225.5 -> 0.00 mm
- net +5V: track 270.4 -> 62.9 mm
- net key_row5: track 164.4 -> 0.00 mm
- net key_col3: track 79.2 -> 0.00 mm
- net key_col2: track 67.1 -> 0.00 mm
- net key_row6: track 66.3 -> 0.00 mm
- net key_row7: track 63.6 -> 0.00 mm
- net key_row3: track 52.5 -> 0.00 mm
- net key_row2: track 41.0 -> 0.00 mm
- net I2C_SDA: track 37.0 -> 0.00 mm
- net I2C_SCL: track 36.4 -> 0.00 mm
- net Net-(D11-A): track 18.2 -> 0.00 mm
- net Net-(D12-A): track 17.6 -> 0.00 mm
- net Net-(D8-A): track 14.9 -> 0.00 mm
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Other:
- board text added: "+ -"
- board text added: "Designed with <3 by Andrew Jia"
- board text added: "LITE"
- board text added: "M7LZY"
- board text added: "STAR"
- board text added: "aka {dblquote}Captain Moonlite{dblquote}"
- board text added: "who received invaluable assistance from SHUBH and Princess Sua"

Commit message: routed central board
Parts:
- moved BT1 14.5 mm to (145.0, 320.5)
- moved C1 14.5 mm to (120.0, 179.5)
- moved C2 14.5 mm to (126.5, 160.0)
- moved C3 14.5 mm to (133.0, 269.0)
- moved C4 14.5 mm to (138.3, 268.0)
- moved D1 14.5 mm to (124.5, 123.1)
- moved D10 14.5 mm to (129.3, 154.1)
- moved D11 14.5 mm to (156.5, 179.8)
- moved D12 14.5 mm to (129.9, 203.4)
- moved D13 14.5 mm to (135.9, 213.9)
- moved D14 14.5 mm to (131.9, 242.4)
- moved D15 14.5 mm to (204.1, 132.6)
- moved D16 14.5 mm to (204.1, 127.6)
- moved D17 14.5 mm to (204.1, 137.6)
- moved D18 14.5 mm to (206.0, 175.7)
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
Commit message: rearranged to fix clearance and alignment
Parts:
- removed BT1: Battery, digisax_stuff:5V0_terminal
- added thumb1: MountingHole_3.2mm_M3, MountingHole:MountingHole_3.2mm_M3, F.Cu at (145.5, 206.0)
- added thumb2: MountingHole_3.2mm_M3, MountingHole:MountingHole_3.2mm_M3, F.Cu at (145.5, 253.0)
- moved U1 75.4 mm to (176.0, 321.3), turned to 90 degrees
- moved J9 49.0 mm to (182.0, 316.0), turned to 180 degrees
- moved SW1 31.9 mm to (183.0, 283.0)
- moved J4 19.9 mm to (168.0, 195.0)
- moved h1 9.51 mm to (168.5, 95.0)
- moved h3 9.50 mm to (168.5, 154.5)
- moved h4 3.54 mm to (168.5, 166.0)
- moved h9 2.55 mm to (180.5, 95.0)
- moved h11 2.50 mm to (180.5, 154.5)
- moved h5 2.12 mm to (118.5, 206.0)
- moved D15 2.00 mm to (202.1, 132.6)
- moved D16 2.00 mm to (202.1, 127.6)
- moved D17 2.00 mm to (202.1, 137.6)
- moved J1 2.00 mm to (180.5, 130.2)
- moved key_Lside1 2.00 mm to (226.8, 128.1)
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Other:
- board size 160 x 250 mm -> 158 x 250 mm
- board text added: "5V regulated"
- board text removed: "+ -"
