File: starlite_production_pcb/starlite_production_pcb.kicad_pcb (KiCad board)
At the start: 2 copper layers, 103 x 250 mm, 45 parts, among them J2 Conn_01x04_Pin, J4 Conn_01x05_Pin, J6 Conn_01x04_Pin, J8 Conn_01x03_Pin, J9 Barrel_Jack, SW1 RotaryEncoder_Switch, U1 ER_OLEDM0.91_1x-I2C, U2 MPXV7007, U3 MCP3221, U4 TLV320DAC3100_breakout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

Commit message: exported pcb step
Parts:
- added D15: 1N4148, Diode_THT:D_DO-35_SOD27_P7.62mm_Horizontal, F.Cu at (207.6, 121.6)
- added D16: 1N4148, Diode_THT:D_DO-35_SOD27_P7.62mm_Horizontal, F.Cu at (207.6, 116.6)
- added D17: 1N4148, Diode_THT:D_DO-35_SOD27_P7.62mm_Horizontal, F.Cu at (207.6, 126.6)
- added D18: 1N4148, Diode_THT:D_DO-35_SOD27_P7.62mm_Horizontal, F.Cu at (209.5, 164.7)
- added D19: 1N4148, Diode_THT:D_DO-35_SOD27_P7.62mm_Horizontal, F.Cu at (216.5, 202.0)
- added D2: 1N4148, Diode_THT:D_DO-35_SOD27_P7.62mm_Horizontal, F.Cu at (114.5, 143.5)
- added D20: 1N4148, Diode_THT:D_DO-35_SOD27_P7.62mm_Horizontal, F.Cu at (182.2, 202.0)
- added D21: 1N4148, Diode_THT:D_DO-35_SOD27_P7.62mm_Horizontal, F.Cu at (193.3, 202.2)
- added D3: 1N4148, Diode_THT:D_DO-35_SOD27_P7.62mm_Horizontal, F.Cu at (108.3, 147.5)
- added D4: 1N4148, Diode_THT:D_DO-35_SOD27_P7.62mm_Horizontal, F.Cu at (108.3, 169.5)
- added D5: 1N4148, Diode_THT:D_DO-35_SOD27_P7.62mm_Horizontal, F.Cu at (85.3, 255.7)
- added D6: 1N4148, Diode_THT:D_DO-35_SOD27_P7.62mm_Horizontal, F.Cu at (85.3, 259.2)
- added J1: Conn_01x04_Pin, digisax_stuff:pad_1x4, F.Cu at (186.0, 119.2)
- added J3: Conn_01x05_Pin, digisax_stuff:pad_1x5, F.Cu at (184.1, 179.8)
- added J5: Conn_01x04_Pin, digisax_stuff:pad_1x4, F.Cu at (114.3, 175.2)
- added J7: Conn_01x03_Pin, digisax_stuff:pad_1x3, F.Cu at (86.9, 277.7)
- added h10: MountingHole_3.2mm_M3, MountingHole:MountingHole_3.2mm_M3, F.Cu at (237.5, 84.5)
- added h11: MountingHole_3.2mm_M3, MountingHole:MountingHole_3.2mm_M3, F.Cu at (186.5, 143.5)
- added h12: MountingHole_3.2mm_M3, MountingHole:MountingHole_3.2mm_M3, F.Cu at (237.5, 143.5)
- added h13: MountingHole_3.2mm_M3, MountingHole:MountingHole_3.2mm_M3, F.Cu at (184.5, 155.5)
- added h14: MountingHole_3.2mm_M3, MountingHole:MountingHole_3.2mm_M3, F.Cu at (219.5, 155.5)
- added h16: MountingHole_3.2mm_M3, MountingHole:MountingHole_3.2mm_M3, F.Cu at (218.5, 210.5)
- added h17: MountingHole_3.2mm_M3, MountingHole:MountingHole_3.2mm_M3, F.Cu at (184.5, 210.5)
- added h18: MountingHole_3.2mm_M3, MountingHole:MountingHole_3.2mm_M3, F.Cu at (94.5, 122.5)
- added h19: MountingHole_3.2mm_M3, MountingHole:MountingHole_3.2mm_M3, F.Cu at (112.5, 122.5)
- added h20: MountingHole_3.2mm_M3, MountingHole:MountingHole_3.2mm_M3, F.Cu at (94.5, 193.5)
- added h21: MountingHole_3.2mm_M3, MountingHole:MountingHole_3.2mm_M3, F.Cu at (112.5, 193.5)
- added h22: MountingHole_3.2mm_M3, MountingHole:MountingHole_3.2mm_M3, F.Cu at (87.0, 248.5)
- added h23: MountingHole_3.2mm_M3, MountingHole:MountingHole_3.2mm_M3, F.Cu at (112.0, 248.5)
- added h24: MountingHole_3.2mm_M3, MountingHole:MountingHole_3.2mm_M3, F.Cu at (87.0, 292.5)
- added h25: MountingHole_3.2mm_M3, MountingHole:MountingHole_3.2mm_M3, F.Cu at (113.0, 292.5)
- added h9: MountingHole_3.2mm_M3, MountingHole:MountingHole_3.2mm_M3, F.Cu at (186.5, 84.5)
- added key_C1: SW_Push, digisax_stuff:slim_switch, F.Cu at (102.1, 278.6)
- added key_Csharp1: SW_Push, digisax_stuff:slim_switch, F.Cu at (209.0, 184.8)
- added key_Dsharp1: SW_Push, digisax_stuff:slim_switch, F.Cu at (105.1, 260.9)
- added key_Gsharp1: SW_Push, digisax_stuff:slim_switch, F.Cu at (197.0, 170.9)
- added key_LB1: SW_Push, digisax_stuff:slim_switch, F.Cu at (193.1, 189.0)
- added key_LBflat1: SW_Push, digisax_stuff:slim_switch, F.Cu at (205.1, 202.9)
- added key_Lside1: SW_Push, digisax_stuff:slim_switch, F.Cu at (232.3, 117.1)
- added key_Lside2: SW_Push, digisax_stuff:slim_switch, F.Cu at (204.3, 99.1)
- added key_Lside3: SW_Push, digisax_stuff:slim_switch, F.Cu at (192.3, 131.1)
- added key_Rside1: SW_Push, digisax_stuff:slim_switch, F.Cu at (103.1, 136.5)
- added key_Rside2: SW_Push, digisax_stuff:slim_switch, F.Cu at (103.1, 158.5)
- added key_Rside3: SW_Push, digisax_stuff:slim_switch, F.Cu at (103.0, 180.5)
Routing:
- net Net-(J1-Pin_4): track 0.00 -> 77.1 mm
- net Net-(J5-Pin_4): track 0.00 -> 64.8 mm
- net Net-(J3-Pin_5): track 0.00 -> 61.1 mm
- net Net-(D19-K): track 0.00 -> 49.1 mm
- net Net-(D16-K): track 0.00 -> 35.2 mm
- net Net-(J7-Pin_3): track 0.00 -> 35.1 mm
- net Net-(D21-K): track 0.00 -> 35.0 mm
- net Net-(D20-K): track 0.00 -> 32.2 mm
- net Net-(D15-K): track 0.00 -> 28.1 mm
- net Net-(D15-A): track 0.00 -> 27.5 mm
- net Net-(D18-K): track 0.00 -> 26.6 mm
- net Net-(D17-K): track 0.00 -> 26.5 mm
- net Net-(D16-A): track 0.00 -> 26.1 mm
- net Net-(D17-A): track 0.00 -> 23.0 mm
- net Net-(D20-A): track 0.00 -> 21.7 mm
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Other:
- board size 103 x 250 mm -> 158.5 x 250 mm

Commit message: routed new pcb
Parts:
- removed BT1: Battery, digisax_stuff:5V0_terminal
- added thumb1: MountingHole_3.2mm_M3, MountingHole:MountingHole_3.2mm_M3, F.Cu at (149.5, 203.5)
- added thumb2: MountingHole_3.2mm_M3, MountingHole:MountingHole_3.2mm_M3, F.Cu at (149.5, 250.5)
- moved U1 83.6 mm to (180.0, 318.8), turned to 90 degrees
- moved J9 50.3 mm to (186.0, 313.5), turned to 180 degrees
- moved SW1 39.0 mm to (187.0, 280.5)
- moved J4 18.0 mm to (172.0, 192.5)
- moved h3 13.1 mm to (172.5, 152.0)
- moved h1 12.8 mm to (172.5, 92.5)
- moved h20 10.2 mm to (92.7, 203.5)
- moved h5 10.0 mm to (122.5, 203.5)
- moved h21 10.0 mm to (111.7, 203.5)
- moved h16 9.16 mm to (220.2, 219.5)
- moved h24 9.09 mm to (85.7, 301.5)
- moved h25 9.09 mm to (111.7, 301.5)
- moved h6 9.06 mm to (172.5, 219.5)
- moved h17 9.00 mm to (184.7, 219.5)
- moved h8 9.00 mm to (122.5, 301.5)
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Routing:
- net EC11_button: track 54.4 -> 9.82 mm, vias 1 -> 0
- net key_row4: track 175.2 -> 143.2 mm
- net EC11_A: track 47.2 -> 19.5 mm, vias 1 -> 0
- net key_row5: track 155.3 -> 179.1 mm, vias 1 -> 0
- net key_row7: track 110.1 -> 132.8 mm, vias 1 -> 2
- net EC11_B: track 37.6 -> 14.8 mm
- net I2C_SCL: track 193.6 -> 175.8 mm, vias 2 -> 1
- net key_row3: track 202.6 -> 219.2 mm, vias 1 -> 2
- net I2C_SDA: track 183.4 -> 199.9 mm
- net key_row6: track 150.2 -> 165.1 mm, vias 0 -> 2
- net GND: track 330.2 -> 315.7 mm, vias 0 -> 3
- net key_col3: track 157.9 -> 169.2 mm
- net +3.3V: track 39.8 -> 49.3 mm
- net key_col2: track 218.5 -> 211.6 mm, vias 3 -> 2
- net +5V: track 235.4 -> 230.1 mm, vias 2 -> 4
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Other:
- board size 158.5 x 250 mm -> 158 x 250 mm
- board text added: "5V regulated"
- board text added: "MountingHole_3.2mm_M3"
- board text removed: "+ -"
