File: starlite_production_pcb/starlite_production_pcb.kicad_pcb (KiCad board)
At the start: 2 copper layers, 158 x 250 mm, 90 parts, among them J1 Conn_01x04_Pin, J2 Conn_01x04_Pin, J3 Conn_01x05_Pin, J4 Conn_01x05_Pin, J5 Conn_01x04_Pin, J6 Conn_01x04_Pin, J7 Conn_01x03_Pin, J8 Conn_01x03_Pin, J9 Barrel_Jack, SW1 RotaryEncoder_Switch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

Commit message: added mouse bites to startlite_production_pcb
Parts:
- added mouse-bite-2.54mm-slot: VAL**, mouse_bites:mouse-bite-2.54mm-slot, F.Cu at (117.7, 140.2)
- added mouse-bite-2.54mm-slot: VAL**, mouse_bites:mouse-bite-2.54mm-slot, F.Cu at (177.3, 169.9)
- added mouse-bite-2.54mm-slot: VAL**, mouse_bites:mouse-bite-2.54mm-slot, F.Cu at (177.4, 103.5)
- added mouse-bite-2.54mm-slot: VAL**, mouse_bites:mouse-bite-2.54mm-slot, F.Cu at (117.7, 294.1)
- added mouse-bite-2.54mm-slot: VAL**, mouse_bites:mouse-bite-2.54mm-slot, F.Cu at (117.7, 195.1)
- added mouse-bite-2.54mm-slot: VAL**, mouse_bites:mouse-bite-2.54mm-slot, F.Cu at (177.4, 141.2)
- added mouse-bite-2.54mm-slot: VAL**, mouse_bites:mouse-bite-2.54mm-slot, F.Cu at (201.2, 158.7)
- added mouse-bite-2.54mm-slot: VAL**, mouse_bites:mouse-bite-2.54mm-slot, F.Cu at (117.7, 262.8)
- added mouse-bite-2.54mm-slot: VAL**, mouse_bites:mouse-bite-2.54mm-slot, F.Cu at (177.3, 213.4)
- moved D15 3.16 mm to (203.7, 131.9)
- moved D16 3.16 mm to (203.7, 126.9)
- moved D17 3.16 mm to (203.7, 136.9)
- moved J1 3.16 mm to (182.1, 129.6)
- moved h11 3.16 mm to (182.1, 153.8)
- moved h12 3.16 mm to (234.1, 153.8)
- moved key_Lside1 3.16 mm to (228.4, 127.4)
- moved key_Lside2 3.16 mm to (200.4, 109.4)
- moved key_Lside3 3.16 mm to (188.4, 141.4)
- moved h10 3.16 mm to (234.1, 94.3)
- moved h9 3.16 mm to (182.1, 94.3)
- moved J3 2.60 mm to (182.2, 188.3)
- moved key_Gsharp1 2.60 mm to (195.1, 179.4)
- moved D18 2.60 mm to (207.6, 173.2)
- moved D19 2.60 mm to (214.6, 210.5)
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Other:
- board size 158 x 250 mm -> 154.2 x 250 mm
